File: Schematic.brd (EAGLE design)
At the start: 100 x 80 mm, 12 parts, among them IC1 MEGA8-AI, IC2 MCP1700 3302E, J1 DCJ0202

Commit message: More components
Parts:
- removed C1: 0.33nF, eagle-ltspice:C1608
- removed C2, C3: 100nF, eagle-ltspice:C1608
- removed IC2: MCP1700 3302E, adafruit:TO92-INLINE
- removed U$1: DS3231, DS3231:SO16
- added POWER_SUPPLY1:C1: 0.33nF, eagle-ltspice:C1608
- added POWER_SUPPLY1:C2, POWER_SUPPLY1:C3: 100nF, eagle-ltspice:C1608
- added POWER_SUPPLY1:IC2: MCP1700 3302E, adafruit:TO92-INLINE
- added RTC1:BACKUP_BAT: CR03N, battery:CR03N
- added RTC1:C1, RTC1:C2: (no value), rcl:SMC_C
- added RTC1:IC1: (no value), DS3231_industrialberry:SOIC-16W
- added RTC1:R1, RTC1:R2: (no value), resistor:M1206
- added SD1:R1: 10k, rcl:M1206
- added SD1:U$1: SDMMC18650, adafruit:SDCARD
- moved IC1 24.2 mm to (29.2, 41.9)
Connections:
- removed net N$3 (its old number): C2.1, IC2.2, J1.3
- new net GND: IC1.5, J1.1, JP1.1, JP1.2, R1.1, RESET.4, RTC1:BACKUP_BAT.-, RTC1:C1.-, RTC1:C2.-, RTC1:IC1.10, RTC1:IC1.11, RTC1:IC1.12, RTC1:IC1.13, RTC1:IC1.5, RTC1:IC1.6, RTC1:IC1.7, RTC1:IC1.8, RTC1:IC1.9, WAKE_UP.4
- new net N$10: IC1.27, RTC1:R2.2
- new net N$2: J1.3, POWER_SUPPLY1:C2.1, POWER_SUPPLY1:IC2.2
- new net N$9: IC1.28, RTC1:R1.2
- new net RTC1:32KHZ: RTC1:IC1.1
- new net RTC1:N$1: RTC1:IC1.15, RTC1:R2.1
- new net RTC1:N$2: RTC1:IC1.16, RTC1:R1.1
- new net RTC1:VBAT: RTC1:BACKUP_BAT.+, RTC1:C1.+, RTC1:IC1.14
- new net SD1:CD: SD1:R1.1
- new net SD1:CS: SD1:U$1.1
- new net SD1:GND: SD1:U$1.COM, SD1:U$1.MT1
- new net SD1:MISO: SD1:U$1.7
- new net SD1:MOSI: SD1:U$1.2
- new net SD1:SCK: SD1:U$1.5
- new net SD1:VCC: SD1:R1.2, SD1:U$1.3, SD1:U$1.6
- new net SD1:WRITE_PROTECT: SD1:U$1.WP
- net N$1: now also RTC1:IC1.3
- net N$7: now also POWER_SUPPLY1:C1.2, POWER_SUPPLY1:C2.2, POWER_SUPPLY1:C3.2, POWER_SUPPLY1:IC2.1; no longer C1.2, C2.2, C3.2, IC1.5, IC2.1, J1.1, JP1.1, JP1.2, R1.1, RESET.4, U$1.10, U$1.11, U$1.12, U$1.13, U$1.5, U$1.6, U$1.7, U$1.8, U$1.9, WAKE_UP.4
- net VCC: now also POWER_SUPPLY1:C1.1, POWER_SUPPLY1:C3.1, POWER_SUPPLY1:IC2.3, RTC1:C2.+, RTC1:IC1.2; no longer C1.1, C3.1, IC2.3

Commit message: More development
Parts:
- removed SD1:R1: 10k, rcl:M1206
- added 1WIRE1:JP1: (no value), pinhead:1X03/90
- added 1WIRE1:R2: 4,7k, resistor:R1206
- added D1: (no value), diode:DO214AA
- added Q1: IRLML5203, transistor-power:MICRO3
- added R2, R3: 10k, rcl:R1206
- added SD1:R2: 10k, rcl:M1206
- added VIZ1:D1: SFH206, opto-trans-siemens:SFH206
- added VIZ1:IC1: LM358D, linear:SO08
- added VIZ1:LED1: (no value), adafruit:LED5MM
- added VIZ1:R1: 1M, rcl:R1206
- added VIZ1:R2: 22k, rcl:R1206
- added VIZ1:R3: 180k, rcl:R1206
- added VIZ1:R4: (no value), rcl:R1206
- added VIZ1:U1: 52207-0485, Molex_By_element14_Batch_1:MOLEX_52207-0485
Connections:
- net N$4 renamed VCC5V
- net N$5 renamed DTR
- net N$6 renamed RX
- net N$8 renamed TX
- removed net SD1:CD: SD1:R1.1
- removed net SD1:CS: SD1:U$1.1
- removed net SD1:GND: SD1:U$1.COM, SD1:U$1.MT1
- removed net SD1:MOSI: SD1:U$1.2
- removed net SD1:VCC: SD1:R1.2, SD1:U$1.3, SD1:U$1.6
- new net N$1: IC1.9, Q1.1
- new net N$11: IC1.16
- new net N$12: IC1.15, SD1:U$1.2
- new net N$13: IC1.17
- new net N$14: IC1.14, SD1:R2.1, SD1:U$1.1
- new net N$16: 1WIRE1:JP1.2, 1WIRE1:R2.1, IC1.12
- new net N$17: D1.C, R2.1, R3.1
- new net N$18: IC1.23, VIZ1:R4.2, VIZ1:U1.2
- new net N$19: IC1.24, VIZ1:IC1.1, VIZ1:R3.2
- new net VIZ1:N$1: VIZ1:D1.K, VIZ1:IC1.2, VIZ1:R1.1
- new net VIZ1:N$2: VIZ1:LED1.A, VIZ1:R4.1
- new net VIZ1:N$3: VIZ1:IC1.3, VIZ1:R2.2, VIZ1:R3.1
- new net VSS_SWITCHED: 1WIRE1:JP1.1, 1WIRE1:R2.2, D1.A, Q1.3
- net GND: now also 1WIRE1:JP1.3, SD1:U$1.COM, SD1:U$1.MT1, VIZ1:D1.A, VIZ1:IC1.4, VIZ1:LED1.K, VIZ1:R2.1, VIZ1:U1.4, VIZ1:U1.5, VIZ1:U1.6
- net N$10: now also R2.2
- net N$9: now also R3.2
- net VCC: now also Q1.2, SD1:R2.2, SD1:U$1.3, SD1:U$1.6, VIZ1:IC1.8, VIZ1:R1.2

Commit message: Slight changes
Connections:
- net N$3 renamed RESET
- net GND: now also IC1.3
Changed lines of the file:
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@@
 <wire x1="3.81" y1="64.77" x2="16.93" y2="62.23" width="0" layer="19" extent="1-1"/>
 </signal>
-<signal name="N$3">
+<signal name="RESET">
 <contactref element="RESET" pad="2"/>
 <contactref element="R1" pad="2"/>
@@
 <contactref element="JP1" pad="1"/>
 <contactref element="J1" pad="1"/>
-<contactref element="WAKE_UP" pad="4"/>
-<contactref element="IC1" pad="5"/>
-<contactref element="RESET" pad="4"/>
-<contactref element="R1" pad="1"/>
 <contactref element="JP1" pad="2"/>
 <contactref element="RTC1:IC1" pad="5"/>
@@
 <contactref element="VIZ1:U1" pad="5"/>
 <contactref element="VIZ1:U1" pad="4"/>
+<contactref element="RESET" pad="4"/>
+<contactref element="R1" pad="1"/>
+<contactref element="IC1" pad="3"/>
+<contactref element="IC1" pad="5"/>
+<contactref element="WAKE_UP" pad="4"/>
 <wire x1="88.9" y1="59.69" x2="88.265" y2="65.98" width="0" layer="19" extent="1-1"/>
 <wire x1="76.2" y1="66.04" x2="88.265" y2="65.98" width="0" layer="19" extent="1-1"/>
@@
 <wire x1="27.94" y1="31.115" x2="38.14" y2="22.86" width="0" layer="19" extent="1-1"/>
 <wire x1="24.9174" y1="41.51" x2="27.94" y2="31.115" width="0" layer="19" extent="1-1"/>
+<wire x1="24.9174" y1="43.11" x2="24.9174" y2="41.51" width="0" layer="19" extent="1-1"/>
 <wire x1="15.24" y1="26.518" x2="27.94" y2="31.115" width="0" layer="19" extent="1-1"/>
 <wire x1="9.6012" y1="25.6794" x2="15.24" y2="26.518" width="0" layer="19" extent="1-1"/>
@@
 <wire x1="48.0314" y1="4.8006" x2="54.1782" y2="7.1374" width="0" layer="19" extent="1-1"/>
 <wire x1="44.8818" y1="7.1374" x2="48.0314" y2="4.8006" width="0" layer="19" extent="1-1"/>
-<wire x1="1.98" y1="55.88" x2="24.9174" y2="41.51" width="0" layer="19" extent="1-1"/>
+<wire x1="1.98" y1="55.88" x2="24.9174" y2="43.11" width="0" layer="19" extent="1-1"/>
 <wire x1="3.81" y1="74.93" x2="1.98" y2="55.88" width="0" layer="19" extent="1-1"/>
 <wire x1="3.81" y1="77.47" x2="3.81" y2="74.93" width="0" layer="19" extent="1-1"/>
