File: Schematic.sch (EAGLE design)
At the start: 12 parts, among them IC1 MEGA8-AI, IC2 MCP1700 3302E, J1 DCJ0202

Commit message: More components
Parts:
- removed C1: 0.33nF, eagle-ltspice:CC1608
- removed C2, C3: 100nF, eagle-ltspice:CC1608
- removed IC2: MCP1700 3302E, adafruit:MCP1700INLINE
- removed U$1: DS3231, DS3231:DS3231
Connections:
- removed net N$3 (its old number): C2.1, IC2.IN, J1.3
- removed net N$7: C1.2, C2.2, C3.2, IC1.GND@2, IC2.GND, J1.1, JP1.1, JP1.2, R1.1, RESET.P1, U$1.GND, U$1.P$1, U$1.P$2, U$1.P$3, U$1.P$4, U$1.P$5, U$1.P$6, U$1.P$7, U$1.P$8, WAKE_UP.P1
- new net 32KHZ: IC1.32KHZ
- new net CD: R1.1
- new net GND: IC1.GND, IC1.GND@2, IC1.NC@1, IC1.NC@2, IC1.NC@3, IC1.NC@4, IC1.NC@5, IC1.NC@6, IC1.NC@7, IC1.NC@8, J1.1, JP1.1, JP1.2, R1.1, RESET.P1, WAKE_UP.P1
- new net INT/SQW: IC1.!INT
- new net N$10: IC1.PC4(ADC4/SDA)
- new net N$2: IC1.SCL, J1.3, R1.1
- new net N$9: IC1.PC5(ADC5/SCL)
- new net SCL: R1.2
- new net VBAT: IC1.VBAT
- net N$1: now also IC1.SDA
- net VCC: now also IC1.VCC, R1.2; no longer C1.1, C3.1, IC2.OUT
Other:
- moved on the sheet: C4

Commit message: More development
Parts:
- added D1: (no value), diode:DIODE-DO214AA
- added Q1: IRLML5203, transistor-power:IRLML5203
- added R2, R3: 10k, rcl:R-EU_R1206
- C4: MF (none) -> AVX; MPN (none) -> 02016D104KAT2A; OC_FARNELL (none) -> 2280755
- IC1, JP1, R1: OC_FARNELL (none) -> unknown
- RESET, WAKE_UP: MF (none) -> OMRON ELECTRONIC COMPONENTS
Connections:
- net N$4 renamed VCC5V
- net N$5 renamed DTR
- net N$6 renamed RX
- net N$8 renamed TX
- removed net CD: R1.1
- new net CS: R2.1
- new net DATA: JP1.2, R2.1
- new net N$11: IC1.PB4(MISO)
- new net N$12: IC1.PB3(MOSI/OC2)
- new net N$13: IC1.PB5(SCK)
- new net N$14: IC1.PB2(SS/OC1B)
- new net N$15: IC1.PD2(INT0), WAKE_UP.S1
- new net N$16: IC1.PB0(ICP)
- new net N$17: D1.C, R2.1, R3.1
- new net N$18: IC1.PC0(ADC0)
- new net N$19: IC1.PC1(ADC1)
- new net OUT: IC1.OUT, R3.2
- new net SDA: R2.2
- new net VSS_SWITCHED: D1.A, Q1.D
- net GND: now also D1.A, IC1.V-, JP1.3, R2.1
- net N$1: now also D1.C, IC1.-IN, IC1.PD5(T1), Q1.G, R1.1, R2.1; no longer IC1.PD2(INT0), WAKE_UP.S1
- net N$10: now also R2.2
- net N$3: now also IC1.+IN, R2.2, R3.1
- net N$9: now also R3.2
- net VCC: now also IC1.V+, JP1.1, Q1.S, R2.2

Commit message: Slight changes
Connections:
- new net RESET: C4.2, IC1.PC6(/RESET), R1.2, RESET.S1
- net GND: now also IC1.GND@1
- net N$3: no longer C4.2, IC1.PC6(/RESET), R1.2, RESET.S1
Other:
- moved on the sheet: R1, RESET
Changed lines of the file:
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@@
 <part name="P+4" library="supply1" deviceset="VCC" device=""/>
 <part name="GND5" library="supply1" deviceset="GND" device=""/>
+<part name="GND6" library="supply1" deviceset="GND" device=""/>
+<part name="GND7" library="supply1" deviceset="GND" device=""/>
+<part name="GND8" library="supply1" deviceset="GND" device=""/>
 </parts>
 <sheets>
@@
 <attribute name="MPN" x="40.64" y="160.02" size="1.778" layer="96" display="off"/>
 </instance>
-<instance part="R1" gate="G$1" x="73.66" y="269.24">
-<attribute name="OC_FARNELL" x="73.66" y="269.24" size="1.778" layer="96" display="off"/>
-<attribute name="MF" x="73.66" y="269.24" size="1.778" layer="96" display="off"/>
-<attribute name="MPN" x="73.66" y="269.24" size="1.778" layer="96" display="off"/>
-</instance>
-<instance part="RESET" gate="1" x="73.66" y="276.86" rot="R270"/>
+<instance part="R1" gate="G$1" x="96.52" y="261.62">
+<attribute name="OC_FARNELL" x="96.52" y="261.62" size="1.778" layer="96" display="off"/>
+<attribute name="MF" x="96.52" y="261.62" size="1.778" layer="96" display="off"/>
+<attribute name="MPN" x="96.52" y="261.62" size="1.778" layer="96" display="off"/>
+</instance>
+<instance part="RESET" gate="1" x="96.52" y="269.24" rot="R270"/>
 <instance part="WAKE_UP" gate="1" x="182.88" y="271.78" rot="R270"/>
 <instance part="P+1" gate="VCC" x="91.44" y="213.36"/>
@@
 <instance part="P+4" gate="VCC" x="109.22" y="271.78" rot="R90"/>
 <instance part="GND5" gate="1" x="109.22" y="279.4" rot="R270"/>
+<instance part="GND6" gate="1" x="104.14" y="226.06" rot="R270"/>
+<instance part="GND7" gate="1" x="88.9" y="251.46" rot="R270"/>
+<instance part="GND8" gate="1" x="172.72" y="269.24" rot="R270"/>
 </instances>
 <busses>
@@
 <pinref part="J1" gate="G$1" pin="2"/>
 <wire x1="30.48" y1="198.12" x2="25.4" y2="198.12" width="0.1524" layer="91"/>
+<label x="30.48" y="175.26" size="1.778" layer="95" xref="yes"/>
 </segment>
 </net>
@@
 <wire x1="170.18" y1="231.14" x2="170.18" y2="170.18" width="0.1524" layer="91"/>
 <wire x1="170.18" y1="170.18" x2="17.78" y2="170.18" width="0.1524" layer="91"/>
+<label x="96.52" y="170.18" size="1.778" layer="95" rot="R270" xref="yes"/>
 </segment>
 </net>
@@
 <wire x1="167.64" y1="172.72" x2="167.64" y2="233.68" width="0.1524" layer="91"/>
 <wire x1="167.64" y1="233.68" x2="154.94" y2="233.68" width="0.1524" layer="91"/>
+<label x="96.52" y="172.72" size="1.778" layer="95" rot="R90" xref="yes"/>
 </segment>
 </net>
@@
 <pinref part="GND1" gate="1" pin="GND"/>
 <wire x1="71.12" y1="182.88" x2="71.12" y2="180.34" width="0.1524" layer="91"/>
-<pinref part="RESET" gate="1" pin="P1"/>
-<pinref part="R1" gate="G$1" pin="1"/>
-<wire x1="68.58" y1="274.32" x2="68.58" y2="269.24" width="0.1524" layer="91"/>
 <wire x1="40.64" y1="180.34" x2="40.64" y2="200.66" width="0.1524" layer="91"/>
 <pinref part="JP1" gate="A" pin="1"/>
@@
 <pinref part="J1" gate="G$1" pin="1"/>
 <wire x1="25.4" y1="200.66" x2="40.64" y2="200.66" width="0.1524" layer="91"/>
-<pinref part="IC1" gate="G$1" pin="GND@2"/>
-<wire x1="22.86" y1="223.52" x2="40.64" y2="223.52" width="0.1524" layer="91"/>
-<wire x1="40.64" y1="223.52" x2="109.22" y2="223.52" width="0.1524" layer="91"/>
-<wire x1="111.76" y1="226.06" x2="22.86" y2="226.06" width="0.1524" layer="91"/>
-<wire x1="22.86" y1="226.06" x2="22.86" y2="223.52" width="0.1524" layer="91"/>
-<wire x1="111.76" y1="251.46" x2="68.58" y2="251.46" width="0.1524" layer="91"/>
-<wire x1="68.58" y1="251.46" x2="33.02" y2="251.46" width="0.1524" layer="91"/>
-<wire x1="33.02" y1="251.46" x2="22.86" y2="251.46" width="0.1524" layer="91"/>
-<wire x1="22.86" y1="251.46" x2="22.86" y2="226.06" width="0.1524" layer="91"/>
-<junction x="22.86" y="226.06"/>
-<wire x1="40.64" y1="200.66" x2="40.64" y2="223.52" width="0.1524" layer="91"/>
-<junction x="40.64" y="200.66"/>
-<junction x="40.64" y="223.52"/>
-<wire x1="68.58" y1="269.24" x2="68.58" y2="251.46" width="0.1524" layer="91"/>
-<junction x="68.58" y="269.24"/>
-<junction x="68.58" y="251.46"/>
-<pinref part="WAKE_UP" gate="1" pin="P1"/>
-<wire x1="177.8" y1="269.24" x2="177.8" y2="287.02" width="0.1524" layer="91"/>
-<wire x1="177.8" y1="287.02" x2="33.02" y2="287.02" width="0.1524" layer="91"/>
-<wire x1="33.02" y1="287.02" x2="33.02" y2="251.46" width="0.1524" layer="91"/>
-<junction x="33.02" y="251.46"/>
 <wire x1="40.64" y1="180.34" x2="71.12" y2="180.34" width="0.1524" layer="91"/>
 <junction x="40.64" y="180.34"/>
@@
 <pinref part="GND5" gate="1" pin="GND"/>
 </segment>
+<segment>
+<wire x1="111.76" y1="251.46" x2="91.44" y2="251.46" width="0.1524" layer="91"/>
+<pinref part="R1" gate="G$1" pin="1"/>
+<pinref part="RESET" gate="1" pin="P1"/>
+<wire x1="91.44" y1="266.7" x2="91.44" y2="261.62" width="0.1524" layer="91"/>
+<junction x="91.44" y="261.62"/>
+<wire x1="91.44" y1="261.62" x2="91.44" y2="251.46" width="0.1524" layer="91"/>
+<pinref part="GND7" gate="1" pin="GND"/>
+<junction x="91.44" y="251.46"/>
+</segment>
+<segment>
+<pinref part="IC1" gate="G$1" pin="GND@1"/>
+<wire x1="109.22" y1="226.06" x2="106.68" y2="226.06" width="0.1524" layer="91"/>
+<pinref part="IC1" gate="G$1" pin="GND@2"/>
+<wire x1="109.22" y1="223.52" x2="106.68" y2="226.06" width="0.1524" layer="91"/>
+<pinref part="GND6" gate="1" pin="GND"/>
+<junction x="106.68" y="226.06"/>
+</segment>
+<segment>
+<pinref part="WAKE_UP" gate="1" pin="P1"/>
+<pinref part="GND8" gate="1" pin="GND"/>
+<wire x1="177.8" y1="269.24" x2="175.26" y2="269.24" width="0.1524" layer="91"/>
+</segment>
 </net>
 <net name="VCC" class="0">
@@
 <pinref part="P+1" gate="VCC" pin="VCC"/>
 <wire x1="91.44" y1="210.82" x2="91.44" y2="200.66" width="0.1524" layer="91"/>
-<wire x1="53.34" y1="218.44" x2="99.06" y2="218.44" width="0.1524" layer="91"/>
+<wire x1="88.9" y1="218.44" x2="99.06" y2="218.44" width="0.1524" layer="91"/>
 <wire x1="99.06" y1="218.44" x2="111.76" y2="218.44" width="0.1524" layer="91"/>
-<wire x1="111.76" y1="220.98" x2="53.34" y2="220.98" width="0.1524" layer="91"/>
-<wire x1="53.34" y1="220.98" x2="53.34" y2="218.44" width="0.1524" layer="91"/>
-<wire x1="111.76" y1="246.38" x2="53.34" y2="246.38" width="0.1524" layer="91"/>
-<wire x1="53.34" y1="246.38" x2="53.34" y2="220.98" width="0.1524" layer="91"/>
-<junction x="53.34" y="220.98"/>
+<wire x1="111.76" y1="220.98" x2="88.9" y2="220.98" width="0.1524" layer="91"/>
+<wire x1="88.9" y1="220.98" x2="88.9" y2="218.44" width="0.1524" layer="91"/>
+<wire x1="111.76" y1="246.38" x2="88.9" y2="246.38" width="0.1524" layer="91"/>
+<wire x1="88.9" y1="246.38" x2="88.9" y2="220.98" width="0.1524" layer="91"/>
+<junction x="88.9" y="220.98"/>
 <wire x1="91.44" y1="200.66" x2="99.06" y2="200.66" width="0.1524" layer="91"/>
 <wire x1="99.06" y1="200.66" x2="99.06" y2="218.44" width="0.1524" layer="91"/>
@@
 </segment>
 </net>
-<net name="N$3" class="0">
+<net name="RESET" class="0">
 <segment>
 <pinref part="R1" gate="G$1" pin="2"/>
 <pinref part="RESET" gate="1" pin="S1"/>
-<wire x1="78.74" y1="274.32" x2="78.74" y2="269.24" width="0.1524" layer="91"/>
+<wire x1="101.6" y1="266.7" x2="101.6" y2="261.62" width="0.1524" layer="91"/>
 <pinref part="IC1" gate="G$1" pin="PC6(/RESET)"/>
-<wire x1="109.22" y1="256.54" x2="78.74" y2="256.54" width="0.1524" layer="91"/>
-<wire x1="78.74" y1="256.54" x2="78.74" y2="269.24" width="0.1524" layer="91"/>
-<junction x="78.74" y="269.24"/>
+<wire x1="109.22" y1="256.54" x2="101.6" y2="256.54" width="0.1524" layer="91"/>
+<wire x1="101.6" y1="256.54" x2="101.6" y2="261.62" width="0.1524" layer="91"/>
+<junction x="101.6" y="261.62"/>
+<wire x1="101.6" y1="256.54" x2="99.06" y2="256.54" width="0.1524" layer="91"/>
+<junction x="101.6" y="256.54"/>
+<label x="99.06" y="256.54" size="1.778" layer="95" rot="R180" xref="yes"/>
+</segment>
+<segment>
 <pinref part="C4" gate="G$1" pin="2"/>
-<wire x1="45.72" y1="160.02" x2="45.72" y2="256.54" width="0.1524" layer="91"/>
-<wire x1="45.72" y1="256.54" x2="78.74" y2="256.54" width="0.1524" layer="91"/>
-<junction x="78.74" y="256.54"/>
+<wire x1="45.72" y1="160.02" x2="50.8" y2="160.02" width="0.1524" layer="91"/>
+<label x="50.8" y="160.02" size="1.778" layer="95" xref="yes"/>
 </segment>
 </net>
@@
 <pinref part="Q1" gate="G$1" pin="D"/>
 <wire x1="185.42" y1="187.96" x2="185.42" y2="185.42" width="0.1524" layer="91"/>
-<label x="177.8" y="185.42" size="1.778" layer="95"/>
 <portref moduleinst="1WIRE1" port="VCC"/>
 <wire x1="210.82" y1="185.42" x2="190.5" y2="185.42" width="0.1524" layer="91"/>
@@
 <wire x1="190.5" y1="220.98" x2="190.5" y2="185.42" width="0.1524" layer="91"/>
 <junction x="190.5" y="185.42"/>
-</segment>
-</net>
+<label x="182.88" y="185.42" size="1.778" layer="95" rot="R180" xref="yes"/>
+<wire x1="185.42" y1="185.42" x2="182.88" y2="185.42" width="0.1524" layer="91"/>
+<junction x="185.42" y="185.42"/>
+</segment>
+</net>
