File: DataLogger/Schematic.sch (EAGLE design)
At the start: 11 parts, among them IC1 MEGA8-AI, J1 DCJ0202, Q1 IRLML5203

Commit message: Updated layout
Connections:
- net N$11 renamed MISO
- net N$12 renamed MOSI
- net N$13 renamed SCK
- removed net N$14: IC1.PB2(SS/OC1B)
- removed net N$3 (its old number): IC1.+IN, R2.2, R3.1
- removed net OUT: IC1.OUT, R3.2
- new net N$18: IC1.ADC7
- new net N$5: IC1.PC2(ADC2)
- new net N$6: IC1.PC3(ADC3)
- new net N$8: IC1.ADC6
- net 32KHZ: now also R3.1
- net CS: now also IC1.PB2(SS/OC1B)
- net GND: now also IC1.AGND; no longer D1.A, IC1.V-, R2.1
- net N$1: no longer D1.C, IC1.-IN, IC1.SDA, R1.1, R2.1
- net N$2: no longer IC1.SCL, R1.1
- net SCL: now also IC1.SCL, R1.1; no longer R1.2
- net SDA: now also IC1.SDA, R2.1; no longer R2.2
- net TX: now also IC1.PD0(RXD)
- net VCC: now also IC1.AVCC, IC1.VCC@1, IC1.VCC@2, R3.2; no longer IC1.V+
Other:
- note added: "v0.1"
- moved on the sheet: R2

Commit message: Rerouted stuff and replaced with better parts.
Parts:
- removed IC1: MEGA8-AI, avr-6:MEGA8-AI
- added C1: 100nF, rcl:C-EUC1206
- added I1: 10nH, Element14Parts:MLF1608E
- added U1: ATMEGA328P-AU, atmel-atmeg328PU:ATMEGA328P-AU
- C4: device eagle-ltspice:CC1608 -> rcl:C-EUC1206
- R1: device resistor:R-EU_R1206 -> rcl:R-EU_R1206; MF (none) -> VISHAY DRALORIC; MPN (none) -> CRCW12061M00FKEA; OC_FARNELL unknown -> 1469968
- R2, R3: MF (none) -> VISHAY DRALORIC; MPN (none) -> CRCW120610K0FKTA; OC_FARNELL unknown -> 1653050
Connections:
- removed net INT/SQW: IC1.!INT
- new net ADC6: U1.ADC6
- new net ADC7: U1.ADC7
- new net AREF: U1.AREF
- new net AVCC: C1.1, I1.2, U1.AVCC
- new net D1: U1.3
- new net D2: U1.4
- new net D3: U1.5
- new net D4: U1.6
- new net D5: U1.7
- new net LED: U1.2
- net 32KHZ: no longer IC1.32KHZ
- net CS: now also U1.PB2/D10; no longer IC1.PB2(SS/OC1B)
- net GND: now also C1.-, C1.2, U1.10, U1.8, U1.9, U1.GND, U1.GND_2, U1.GND_3; no longer IC1.AGND, IC1.GND, IC1.GND@1, IC1.GND@2, IC1.NC@1, IC1.NC@2, IC1.NC@3, IC1.NC@4, IC1.NC@5, IC1.NC@6, IC1.NC@7, IC1.NC@8
- net MISO: now also U1.PB4/MISO/D12; no longer IC1.PB4(MISO)
- net MOSI: now also U1.PB3/MOSI/D11; no longer IC1.PB3(MOSI/OC2)
- net N$1: now also U1.PD5/D5; no longer IC1.PD5(T1)
- net N$10: now also U1.PC4/SDA/A4; no longer IC1.PC4(ADC4/SDA)
- net N$15: now also U1.PD2/INT0/D2; no longer IC1.PD2(INT0)
- net N$16: now also U1.PB0/D8; no longer IC1.PB0(ICP)
- net N$18: now also U1.PD4/D4; no longer IC1.ADC7
- net N$3: now also U1.PC0/A0; no longer IC1.PC0(ADC0)
- net N$4: now also U1.PC1/A1; no longer IC1.PC1(ADC1)
- net N$5: now also U1.PC2/A2; no longer IC1.PC2(ADC2)
- net N$6: now also U1.PC3/A3; no longer IC1.PC3(ADC3)
- net N$8: now also U1.PD3/INT1/D3; no longer IC1.ADC6
- net N$9: now also U1.PC5/SCL/A5; no longer IC1.PC5(ADC5/SCL)
- net RESET: now also U1.PC6/RESET; no longer IC1.PC6(/RESET)
- net RX: now also U1.PD1/TXD/D1; no longer IC1.PD1(TXD)
- net SCK: now also U1.PB5/SCK/D13; no longer IC1.PB5(SCK)
- net SCL: no longer IC1.SCL
- net SDA: no longer IC1.SDA
- net TX: now also U1.PD0/RXD/D0; no longer IC1.PD0(RXD)
- net VBAT: now also C1.+; no longer IC1.VBAT
- net VCC: now also C1.+, I1.1, U1.1, U1.VCC, U1.VCC_2; no longer IC1.AVCC, IC1.VCC, IC1.VCC@1, IC1.VCC@2
Other:
- moved on the sheet: D1, R2, R3

Commit message: Improvements
Parts:
- added D2: (no value), diode:DIODE-DO214AA
- U1: device atmel-atmeg328PU:ATMEGA328P-AU -> Arduino Dev Parts:ATMEGA328P-AU; MF ATMEL -> (none)
Connections:
- removed net ADC6: U1.ADC6
- removed net ADC7: U1.ADC7
- removed net MISO: U1.PB4/MISO/D12
- removed net MOSI: U1.PB3/MOSI/D11
- removed net N$10: R2.2, U1.PC4/SDA/A4
- removed net N$15: U1.PD2/INT0/D2, WAKE_UP.S1
- removed net N$16: U1.PB0/D8
- removed net N$18: U1.PD4/D4
- removed net N$3: U1.PC0/A0
- removed net N$4: U1.PC1/A1
- removed net N$5: U1.PC2/A2
- removed net N$6: U1.PC3/A3
- removed net N$8: U1.PD3/INT1/D3
- removed net N$9: R3.2, U1.PC5/SCL/A5
- removed net SCK: U1.PB5/SCK/D13
- new net A0: U1.A0
- new net A1: U1.A1
- new net A2: U1.A2
- new net A3: U1.A3
- new net A4: R2.2, U1.A4/SDA
- new net A5: R3.2, U1.A5/SCL
- new net D10: U1.D10/~
- new net D11: U1.D11/MOSI/~
- new net D12: U1.D12/MISO
- new net D13: U1.D13/SCK
- new net D8: U1.D8
- net CS: no longer U1.PB2/D10
- net D2: now also U1.D2/INT0, WAKE_UP.S1
- net D3: now also U1.D3/INT1/~
- net D4: now also U1.D4
- net D5: now also Q1.G, U1.D5/~
- net GND: no longer U1.GND_2, U1.GND_3
- net N$1: now also D2.A, J1.3; no longer Q1.G, U1.PD5/D5
- net N$2: now also D2.C; no longer J1.3
- net RESET: now also U1.!RESET; no longer U1.PC6/RESET
- net RX: now also U1.D1/TXD; no longer U1.PD1/TXD/D1
- net TX: now also U1.D0/RXD; no longer U1.PD0/RXD/D0
- net VCC: no longer U1.VCC_2
Other:
- moved on the sheet: C1, I1, R3
