File: Tests/Amplifier.brd (EAGLE design)
At the start: 47 x 28.9 mm, 20 parts

Commit message: Lots of updates
Parts:
- removed OUTPUT: S4B-ZR, con-jst:S4B-ZR
- added GND, SCL, SDA, VCC: LSP10, solpad:LSP10
Connections:
- net GND: now also GND.MP; no longer OUTPUT.4
- net N$11: now also SDA.MP; no longer OUTPUT.2
- net N$4: now also SCL.MP; no longer OUTPUT.3
- net VSS: now also VCC.MP; no longer OUTPUT.1
Routing:
- net VSS: track 82.8 -> 100.6 mm, vias 1 -> 3
- net GND: track 126.1 -> 137.6 mm, vias 0 -> 1
- net VREF: track 44.1 -> 33.4 mm, vias 2 -> 3
- net N$10: track 53.0 -> 44.0 mm
- net N$11: track 13.5 -> 19.7 mm, vias 1 -> 0
- net N$1: track 15.8 -> 21.5 mm
- net N$12: track 17.8 -> 13.1 mm
- net N$7: track 31.7 -> 36.1 mm, vias 2 -> 0
- net N$3: track 12.6 -> 14.9 mm, vias 0 -> 2
- net SIGNAL: track 25.1 -> 23.3 mm
- net N$9: track 33.6 -> 32.1 mm
- net N$6: track 26.3 -> 25.1 mm
- net N$5: track 15.0 -> 16.1 mm
- net N$8: track 9.14 -> 10.1 mm
- net N$2: track 12.7 -> 12.1 mm, vias 2 -> 0
