File: Tests/Amplifier.sch (EAGLE design)
At the start: 20 parts

Commit message: Lots of updates
Parts:
- removed OUTPUT: S4B-ZR, con-jst:S4B-ZR
- added GND, SCL, SDA, VCC: LSP10, solpad:LSP10
Connections:
- net GND: now also GND.MP; no longer OUTPUT-4.1
- net N$11: now also SDA.MP; no longer OUTPUT-2.1
- net N$4: now also SCL.MP; no longer OUTPUT-3.1
- net VSS: now also VCC.MP; no longer OUTPUT-1.1
Other:
- moved on the sheet: C5, R1
Changed lines of the file:
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@@
 <part name="GND6" library="supply1" deviceset="GND" device=""/>
 <part name="ADC" library="Arduino Dev Parts" deviceset="MCP3021" device="A5T-E/OT"/>
-<part name="OUTPUT" library="con-jst" deviceset="?4B-ZR" device="S" value="S4B-ZR"/>
 <part name="C6" library="rcl" deviceset="CPOL-EU" device="SMCB" value="100nF"/>
 <part name="R5" library="rcl" deviceset="R-EU_" device="R1206" value="220R"/>
@@
 <part name="GND4" library="supply1" deviceset="GND" device=""/>
 <part name="U$1" library="Arduino Dev Parts" deviceset="VBT101BH" device=""/>
+<part name="VCC" library="solpad" deviceset="LSP10" device=""/>
+<part name="SDA" library="solpad" deviceset="LSP10" device=""/>
+<part name="SCL" library="solpad" deviceset="LSP10" device=""/>
+<part name="GND" library="solpad" deviceset="LSP10" device=""/>
 </parts>
 <sheets>
@@
 <instance part="SW" gate="ADG755" x="60.96" y="50.8" rot="R180"/>
 <instance part="C1" gate="G$1" x="-2.54" y="58.42" rot="R90"/>
-<instance part="R1" gate="G$1" x="5.08" y="50.8" rot="R90"/>
+<instance part="R1" gate="G$1" x="5.08" y="48.26" rot="R270"/>
 <instance part="R2" gate="G$1" x="-30.48" y="73.66" rot="R180"/>
 <instance part="C2" gate="G$1" x="-30.48" y="81.28" rot="R90"/>
@@
 <instance part="D1" gate="G$1" x="-10.16" y="111.76" rot="R270"/>
 <instance part="R4" gate="G$1" x="-2.54" y="111.76" rot="R90"/>
-<instance part="C5" gate="G$1" x="-2.54" y="99.06" rot="R180"/>
+<instance part="C5" gate="G$1" x="-2.54" y="99.06"/>
 <instance part="VSS5" gate="G$1" x="99.06" y="124.46" rot="R180"/>
 <instance part="GND5" gate="1" x="83.82" y="27.94"/>
 <instance part="GND6" gate="1" x="99.06" y="83.82"/>
 <instance part="ADC" gate="MCP3021" x="111.76" y="106.68"/>
-<instance part="OUTPUT" gate="-1" x="144.78" y="114.3"/>
-<instance part="OUTPUT" gate="-2" x="144.78" y="111.76"/>
-<instance part="OUTPUT" gate="-3" x="144.78" y="109.22"/>
-<instance part="OUTPUT" gate="-4" x="144.78" y="106.68"/>
 <instance part="C6" gate="G$1" x="73.66" y="109.22"/>
 <instance part="R5" gate="G$1" x="-33.02" y="124.46" rot="R270"/>
@@
 <instance part="GND4" gate="1" x="-33.02" y="109.22"/>
 <instance part="U$1" gate="A" x="-45.72" y="58.42" rot="R180"/>
+<instance part="VCC" gate="1" x="142.24" y="114.3" smashed="yes" rot="R270">
+<attribute name="NAME" x="145.034" y="113.411" size="1.778" layer="95"/>
+</instance>
+<instance part="SDA" gate="1" x="142.24" y="111.76" smashed="yes" rot="R270">
+<attribute name="NAME" x="145.034" y="110.871" size="1.778" layer="95"/>
+</instance>
+<instance part="SCL" gate="1" x="142.24" y="109.22" smashed="yes" rot="R270">
+<attribute name="NAME" x="145.288" y="108.331" size="1.778" layer="95"/>
+</instance>
+<instance part="GND" gate="1" x="142.24" y="106.68" smashed="yes" rot="R270">
+<attribute name="NAME" x="145.034" y="105.791" size="1.778" layer="95"/>
+</instance>
 </instances>
 <busses>
@@
 <junction x="17.78" y="88.9"/>
 <pinref part="C5" gate="G$1" pin="2"/>
-<wire x1="-2.54" y1="104.14" x2="5.08" y2="88.9" width="0.1524" layer="91"/>
+<wire x1="-2.54" y1="93.98" x2="5.08" y2="88.9" width="0.1524" layer="91"/>
 <wire x1="5.08" y1="88.9" x2="17.78" y2="88.9" width="0.1524" layer="91"/>
 <pinref part="C4" gate="G$1" pin="1"/>
@@
 <pinref part="GND6" gate="1" pin="GND"/>
 <wire x1="99.06" y1="86.36" x2="99.06" y2="91.44" width="0.1524" layer="91"/>
-<pinref part="OUTPUT" gate="-4" pin="1"/>
 <wire x1="99.06" y1="91.44" x2="99.06" y2="101.6" width="0.1524" layer="91"/>
 <wire x1="99.06" y1="91.44" x2="124.46" y2="91.44" width="0.1524" layer="91"/>
@@
 <wire x1="73.66" y1="104.14" x2="86.36" y2="91.44" width="0.1524" layer="91"/>
 <wire x1="86.36" y1="91.44" x2="99.06" y2="91.44" width="0.1524" layer="91"/>
+<pinref part="GND" gate="1" pin="MP"/>
 </segment>
 <segment>
@@
 <pinref part="R1" gate="G$1" pin="1"/>
 <wire x1="5.08" y1="58.42" x2="10.16" y2="58.42" width="0.1524" layer="91"/>
-<wire x1="5.08" y1="58.42" x2="5.08" y2="45.72" width="0.1524" layer="91"/>
+<wire x1="5.08" y1="58.42" x2="5.08" y2="53.34" width="0.1524" layer="91"/>
 <junction x="5.08" y="58.42"/>
 </segment>
@@
 <pinref part="R1" gate="G$1" pin="2"/>
 <pinref part="C3" gate="G$1" pin="2"/>
-<wire x1="5.08" y1="40.64" x2="5.08" y2="55.88" width="0.1524" layer="91"/>
+<wire x1="5.08" y1="40.64" x2="5.08" y2="43.18" width="0.1524" layer="91"/>
 <label x="5.08" y="43.18" size="1.778" layer="95" xref="yes"/>
 </segment>
@@
 <pinref part="VSS5" gate="G$1" pin="VSS"/>
 <wire x1="99.06" y1="121.92" x2="99.06" y2="119.38" width="0.1524" layer="91"/>
-<pinref part="OUTPUT" gate="-1" pin="1"/>
 <wire x1="99.06" y1="119.38" x2="99.06" y2="111.76" width="0.1524" layer="91"/>
 <wire x1="99.06" y1="119.38" x2="134.62" y2="119.38" width="0.1524" layer="91"/>
@@
 <wire x1="73.66" y1="111.76" x2="81.28" y2="119.38" width="0.1524" layer="91"/>
 <wire x1="81.28" y1="119.38" x2="99.06" y2="119.38" width="0.1524" layer="91"/>
+<pinref part="VCC" gate="1" pin="MP"/>
 </segment>
 </net>
@@
 <junction x="7.62" y="111.76"/>
 <pinref part="C5" gate="G$1" pin="1"/>
-<wire x1="-2.54" y1="96.52" x2="-2.54" y2="106.68" width="0.1524" layer="91"/>
+<wire x1="-2.54" y1="101.6" x2="-2.54" y2="106.68" width="0.1524" layer="91"/>
 <junction x="-2.54" y="106.68"/>
 <pinref part="D1" gate="G$1" pin="C"/>
@@
 <segment>
 <pinref part="ADC" gate="MCP3021" pin="SCL"/>
-<pinref part="OUTPUT" gate="-3" pin="1"/>
 <wire x1="124.46" y1="106.68" x2="137.16" y2="106.68" width="0.1524" layer="91"/>
 <wire x1="137.16" y1="106.68" x2="139.7" y2="109.22" width="0.1524" layer="91"/>
+<pinref part="SCL" gate="1" pin="MP"/>
 </segment>
 </net>
@@
 <segment>
 <pinref part="ADC" gate="MCP3021" pin="SDA"/>
-<pinref part="OUTPUT" gate="-2" pin="1"/>
 <wire x1="124.46" y1="111.76" x2="139.7" y2="111.76" width="0.1524" layer="91"/>
-</segment>
-</net>
+<pinref part="SDA" gate="1" pin="MP"/>
+</segment>
+</net>
